File: 4xmixer/Faceplate/4xmixerFace.kicad_pcb (KiCad board)
At the start: 2 copper layers, 20.3 x 121.9 mm, 11 parts

Commit message: This faceplate was also incredibly wrong.
Parts:
- removed the REF** at (30.5, 131.4)
- removed the REF** at (30.5, 15.9)
- added REF**: MountingHole_3.2mm_M3, MountingHole:MountingHole_3.2mm_M3, F.Cu at (83.8, 153.3)
- added REF**: MountingHole_3.2mm_M3, MountingHole:MountingHole_3.2mm_M3, F.Cu at (83.8, 29.6)
- moved REF** 56.2 mm to (94.0, 120.7)
- moved REF** 56.2 mm to (94.0, 136.0)
- moved REF** 56.2 mm to (88.8, 43.2)
- moved REF** 56.2 mm to (88.9, 58.5)
- moved REF** 56.2 mm to (88.9, 73.7)
- moved REF** 56.2 mm to (88.9, 89.0)
- moved REF** 56.2 mm to (94.0, 105.5)
- moved REF** 56.2 mm to (83.8, 105.5)
- moved REF** 56.2 mm to (83.8, 120.8)
Other:
- board size 20.3 x 121.9 mm -> 20.3 x 128.6 mm
- board text added: "4Mixer"
- board text added: "Gray"
- board text added: "Noise"
- board text removed: "Gray Noise"
- board text removed: "Mixer"
