File: vccg/Main/vccg/vccg.kicad_pcb (KiCad board)
At the start: 2 copper layers, 50.8 x 103.4 mm, 67 parts, among them J1 ChordCV, J10 root, J11 chord1, J2 OctaveCV, J3 MelodyCV, J4 MelodyClock, J5 ChordClock, J6 Conn_02x05_Odd_Even, J7 oled, J8 melody, J9 chord2, M1 RaspberryPiPico, Q1 MMBT3904, Q2 MMBT3904, SW1 Back, SW2 RotaryEncoder_Switch, U1 MCP6002-xSN, U2 MCP6002-xSN, U3 XL1509, U4 MCP4728, U5 LM2904, U6 LM2904

Commit message: add hex inverter to clean up nasty encoder output
Parts:
- added C5: 10n, Capacitor_SMD:C_0603_1608Metric, F.Cu at (240.1, 82.7)
- added C6: 10n, Capacitor_SMD:C_0603_1608Metric, F.Cu at (228.1, 94.4)
- added C7: 10n, Capacitor_SMD:C_0603_1608Metric, F.Cu at (241.8, 95.1)
- added C9: 10n, Capacitor_SMD:C_0603_1608Metric, F.Cu at (234.5, 108.2)
- added U3: 74HC14, Package_SO:SOIC-14_3.9x8.7mm_P1.27mm, F.Cu at (232.9, 100.5)
- L1: footprint SynthStuff:Inductor_SMD-L_SMMS1040 -> Inductor_SMD:L_6.3x6.3_H3
- R8, R9: value 100K -> 10K
- moved R28 26.9 mm to (214.4, 99.8), turned to 180 degrees
- moved R27 25.1 mm to (214.4, 98.3), turned to 180 degrees
- moved R16 15.6 mm to (223.8, 113.8)
- moved R20 15.6 mm to (223.8, 110.8)
- moved R15 15.4 mm to (214.5, 113.9)
- moved R19 15.4 mm to (214.5, 110.8)
- moved U7 15.4 mm to (219.3, 112.2)
- moved R17 15.3 mm to (214.4, 104.5)
- moved R13 15.3 mm to (214.4, 107.6)
- moved R14 15.2 mm to (223.8, 107.7)
- moved R18 15.2 mm to (223.8, 104.6)
- moved U6 15.1 mm to (219.3, 106.3)
- moved U5 12.4 mm to (219.8, 99.2)
- moved C8 8.56 mm to (207.7, 103.0)
- moved D5 8.49 mm to (211.6, 101.5)
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- renumbered C6 to C10, C5 to C8, U3 to U4, U4 to U5, U5 to U6, U6 to U7
Connections:
- M1 pad 16: SDA0 -> unconnected-(M1-Pad16)
- M1 pad 17: SCL0 -> unconnected-(M1-Pad17)
- M1 pad 21: unconnected-(M1-Pad21) -> SDA0
- M1 pad 22: unconnected-(M1-Pad22) -> SCL0
- M1 pad 24: select -> debounceBack
- M1 pad 25: encoderB -> debounceSelect
- M1 pad 26: encoderA -> debounceB
- M1 pad 27: back -> debounceA
- R19 pad 1: Net-(R19-Pad1) -> Net-(R24-Pad2)
- R20 pad 1: Net-(R20-Pad1) -> Net-(R21-Pad2)
- R21 pad 2: Net-(R17-Pad1) -> Net-(R21-Pad2)
- R22 pad 2: Net-(R18-Pad1) -> Net-(R17-Pad1)
- R23 pad 2: Net-(R19-Pad1) -> Net-(R18-Pad1)
- R24 pad 2: Net-(R20-Pad1) -> Net-(R24-Pad2)
- U7 pad 1: Net-(R19-Pad1) -> Net-(R24-Pad2)
- U7 pad 7: Net-(R20-Pad1) -> Net-(R21-Pad2)
Routing:
- net Net-(R20-Pad1): track 47.9 -> 0.00 mm
- net Net-(R18-Pad1): track 71.0 -> 29.6 mm, vias 0 -> 2
- net +3V3: track 240.0 -> 206.1 mm, vias 7 -> 9
- net Net-(R21-Pad2): track 0.00 -> 27.3 mm, vias 0 -> 2
- net +12V: track 101.1 -> 77.0 mm
- net Net-(R24-Pad2): track 0.00 -> 21.0 mm, vias 0 -> 2
- net Net-(R19-Pad1): track 18.6 -> 0.00 mm
- net GND: track 9.47 -> 19.6 mm, vias 20 -> 18
- net debounceBack: track 0.00 -> 9.95 mm
- net Net-(D3-Pad1): track 19.1 -> 11.6 mm
- net encoderB: track 35.5 -> 28.6 mm
- net back: track 18.2 -> 24.5 mm
- net VOUTB: track 22.1 -> 17.1 mm
- net debounceSelect: track 0.00 -> 4.47 mm
- net debounceB: track 0.00 -> 4.47 mm
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Other:
- board text added: "3V3"
- board text added: "GND"
- board text added: "SCL"
- board text added: "SDA"

Commit message: VCCG Version 1.4
Features:
* New hex inverter signal cleanup on the rotary encoder pins
* Layout updates
* MCP6002 footprint changes to match JLCPCB parts availability
* Inductor footprint changes to match JLCPCB parts availability
Parts:
- L1: footprint Inductor_SMD:L_6.3x6.3_H3 -> SynthStuff:Inductor_SMD-CY75-68uh
- U1, U2: footprint Package_SO:MSOP-8_3x3mm_P0.65mm -> Package_SO:SOIC-8_3.9x4.9mm_P1.27mm
- moved D3 5.59 mm to (204.2, 116.7), turned to -90 degrees
- moved U2 4.51 mm to (208.1, 68.8)
- moved U1 2.55 mm to (199.7, 68.8)
- moved L1 2.25 mm to (208.9, 110.2), turned to -90 degrees
Connections:
- U2 pad 1: melody -> Net-(U2-Pad2)
- U2 pad 2: melody -> Net-(U2-Pad2)
- U2 pad 3: Net-(RV3-Pad2) -> GND
- U2 pad 5: GND -> Net-(RV3-Pad2)
- U2 pad 6: Net-(U2-Pad6) -> melody
- U2 pad 7: Net-(U2-Pad6) -> melody
Routing:
- net +3V3: track 206.1 -> 217.4 mm, vias 9 -> 8
- net Net-(U2-Pad2): track 0.00 -> 4.23 mm
- net Net-(U2-Pad6): track 2.88 -> 0.00 mm
- net Net-(RV2-Pad2): track 21.9 -> 24.7 mm
- net octave: track 52.5 -> 54.6 mm
- net GND: track 19.6 -> 17.7 mm
- net Net-(D3-Pad1): track 11.6 -> 9.83 mm
- net chord: track 55.4 -> 56.8 mm
- net Net-(R17-Pad1): track 29.0 -> 30.3 mm
- net Net-(RV1-Pad2): track 15.1 -> 16.0 mm
- net melody: track 30.8 -> 31.6 mm
Other:
- board text added: "v1.4"
- board text removed: "v1.3"
