File: kassuVCA/Channel3-4.sch (KiCad schematic (older format))
At the start: 83 parts

Commit message: WIP 0805 TL072 dual channel
Connections:
- net Level1L renamed Level3L
- net Level1R renamed Level3R
- net Level2L renamed Level4L
- net Level2R renamed Level4R
