File: kassuVCA/Channel4-5.sch (KiCad schematic (older format))
At the start: 64 parts, among them Q401 MMBT3904, Q402 MBT3904DW1, Q403 MBT3904DW1, Q404 MMBT3904, U401 TL072, U402 TL072

Commit message: 4/6 channels, 4 routed
Parts:
- removed Trim2: 100K, Potentiometer_THT:Potentiometer_Bourns_3296W_Vertical, symbol Device:R_POT
- removed mute1: SW_DPDT_x2, MixerFootprints:A-330-6mm-dpdt, symbol Switch:SW_DPDT_x2
- added SW401: SW_DPDT_x2, MixerFootprints:A-330-6mm-dpdt, symbol Switch:SW_DPDT_x2
- added Trim402: 100K, Potentiometer_THT:Potentiometer_Bourns_3296W_Vertical, symbol Device:R_POT
- CV2: value AudioJack2_Switch -> AudioJack2_SwitchT
- renumbered mute2 to SW402, Trim1 to Trim401
Connections:
- net +12V: now also Trim402.1
- net -12V: now also Trim402.3
- net at C401.1, Q401.1 (B), R409.1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: now also SW401.2 (B)
- net at R412.2: now also Trim402.2
- net at R414.2: now also SW401.1 (A)
