File: vccg/VccgLogicBoard/VccgLogicBoard.kicad_sch (KiCad schematic)
At the start: 71 parts, among them J1 ChordCV, J10 root, J11 chord1, J2 OctaveCV, J3 MelodyCV, J4 MelodyClock, J5 ChordClock, J6 Conn_02x05_Odd_Even, J7 oled, J8 melody, J9 chord2, M1 RaspberryPiPico, Q1 MMBT3904, Q2 MMBT3904, SW1 Back, SW2 RotaryEncoder_Switch, U1 MCP6002-xSN, U2 MCP6002-xSN, U3 74HC14, U4 XL1509, U5 MCP4728, U6 LM2904, U7 LM2904

Commit message: Rebuild with 4 mom buttons instead of rotary encoder
Parts:
- removed C9: 10n, Capacitor_SMD:C_0603_1608Metric, symbol Device:C_Small
- removed SW2: RotaryEncoder_Switch, Rotary_Encoder:RotaryEncoder_Alps_EC11E-Switch_Vertical_H20mm_CircularMountingHoles, symbol Device:RotaryEncoder_Switch
- removed U3: 74HC14, Package_SO:SOIC-14_3.9x8.7mm_P1.27mm, symbol 74xx:74HC14
- added C7: 10n, Capacitor_SMD:C_0603_1608Metric, symbol Device:C_Small
- added R13: 100K, Resistor_SMD:R_0603_1608Metric, symbol Device:R_Small_US
- added R7: 1K, Resistor_SMD:R_0603_1608Metric, symbol Device:R_Small_US
- added SW1: Down, Button_Switch_THT:SW_PUSH_6mm_H13mm, symbol Switch:SW_SPST
- added SW2: Up, Button_Switch_THT:SW_PUSH_6mm_H13mm, symbol Switch:SW_SPST
- added SW3: Select, Button_Switch_THT:SW_PUSH_6mm_H13mm, symbol Switch:SW_SPST
- R11: value 1K -> 100K
- R8, R9: value 10K -> 1K
- renumbered C7 to C8, C8 to C9, J11 to J10, J8 to J11, J10 to J8, R7 to R10, R10 to R14, R13 to R15, R14 to R16, R15 to R17, R16 to R18, R17 to R19, R18 to R20, R19 to R21, R20 to R22, R22 to R23, R23 to R24, R24 to R25, R21 to R26, R25 to R27, R26 to R28, R27 to R29, R28 to R30, R29 to R31, SW1 to SW4, U4 to U3, U5 to U4, U6 to U5, U7 to U6
Connections:
- net debounceB is gone; now on net select: M1.26 (GP20)
- net debounceSelect is gone; now on net back: M1.25 (GP19)
- net +3V3: now also R8.1, R7.1; no longer R11.1, R8.2
- net GND: now also C5.2, R11.2, C7.2, R13.2; no longer C5.1
- net chordClock: now also M1.34 (GP28); no longer M1.6 (GP4)
- net melody: now also M1.37 (3v3_EN); no longer M1.34 (GP28)
- net melodyClock: now also M1.35 (ADC_VREF); no longer M1.2 (GP1)
- net select: now also C7.1, R13.1, SW3.2 (B); no longer R12.1
- net debounceA renamed up
- net up: now also C6.1, R12.1, SW2.2 (B)
- net debounceBack renamed down
- net down: now also C5.1, R11.1, SW1.2 (B)
- removed net encoderA: C6.1, R8.1
- net encoderB: no longer names the net of R9.2
- net encoderB: now also SW3.1 (A); no longer C5.2
- new net: R7.2, SW1.1 (A)
- new net: R8.2, SW2.1 (A)
